File: FlashBack_Schematic/FlashBack_Schematic.kicad_sch (KiCad schematic)
At the start: 47 parts, among them Q1 NPN, Q2 NPN, Q3 AO3401A, SW1 SW_Push, SW2 SW_SPDT, U1 HT-CT62, U2 ADXL345, U3 GY-NEO6MV2, U4 74HC595, U5 MAX17048, U6 TP4054, U7 CE6260B33M, U8 Battery

Commit message: kiCad
Connections:
- net 3V3: now also R14.1, R15.1
- net GND: no longer R14.2, R15.2
- net SCL: now also R15.2; no longer R15.1
- net SDA: now also R14.2; no longer R14.1
Other:
- note added: "GNSS"
- note removed: "GPS"
- moved on the sheet: R14, R15
